Commit message: 更改了足端模型，关闭了自身碰撞，学会了稳定低速小跑，没学会速度跟踪

File: resources/robots/mini_cheetah/urdf/mini_cheetah.urdf (robot description, URDF)
Before this commit: robot mini_cheetah, 15 links, 14 joints
Links:
- added link FL_foot, mass 0.001; collision sphere radius=0.020; visual sphere radius=0.020
- added link FR_foot, mass 0.001; collision sphere radius=0.020; visual sphere radius=0.020
- added link RL_foot, mass 0.001; collision sphere radius=0.020; visual sphere radius=0.020
- added link RR_foot, mass 0.001; collision sphere radius=0.020; visual sphere radius=0.020
Joints:
- added joint FL_foot_fixed: type fixed, parent FL_calf, child FL_foot, origin xyz=0 0 -0.19 rpy=0 0 0
- added joint FR_foot_fixed: type fixed, parent FR_calf, child FR_foot, origin xyz=0 0 -0.19 rpy=0 0 0
- added joint RL_foot_fixed: type fixed, parent RL_calf, child RL_foot, origin xyz=0 0 -0.19 rpy=0 0 0
- added joint RR_foot_fixed: type fixed, parent RR_calf, child RR_foot, origin xyz=0 0 -0.19 rpy=0 0 0
